File: router_power_board/router_LiPo.kicad_pcb (KiCad board)
At the start: 2 copper layers, 90 x 45 mm, 32 parts, among them J1 Conn_01x02, J2 Conn_01x02, J4 Conn_01x02, Q1 RS6L120BGTB1, Q2 RS6L120BGTB1, U1 LM5050-1, U2 LM5050-1, U4 TPS54560BDDA

Commit message: add M2.5 hole
Parts:
- added REF**: MountingHole_2.7mm_M2.5, MountingHole:MountingHole_2.7mm_M2.5, F.Cu at (237.0, 79.5)
- added REF**: MountingHole_2.7mm_M2.5, MountingHole:MountingHole_2.7mm_M2.5, F.Cu at (237.0, 40.5)
- added REF**: MountingHole_2.7mm_M2.5, MountingHole:MountingHole_2.7mm_M2.5, F.Cu at (153.0, 79.5)
- added REF**: MountingHole_2.7mm_M2.5, MountingHole:MountingHole_2.7mm_M2.5, F.Cu at (153.0, 40.5)
Routing:
- net GNDD: vias 315 -> 299
